File: 3d_Printer_Interface.sch (KiCad schematic (older format))
At the start: 0 parts

Commit message: Completed Initial Schematic
Parts:
- added J? (x6): Conn_01x03, symbol Connector_Generic:Conn_01x03
- added J?: Conn_01x04, symbol Connector_Generic:Conn_01x04
Connections:
- net MCU/AD0: now also J?.3 (Pin_3)
- net MCU/AD1: now also J?.3 (Pin_3)
- net MCU/AD2: now also J?.3 (Pin_3)
- net MCU/AD3: now also J?.3 (Pin_3)
- net MCU/AD6: now also J?.3 (Pin_3)
- net MCU/AD7: now also J?.3 (Pin_3)
- new net: J?.1 (Pin_1), J?.1 (Pin_1), J?.1 (Pin_1), J?.1 (Pin_1), J?.1 (Pin_1), J?.1 (Pin_1)
- new net +5V: J?.2 (Pin_2), J?.2 (Pin_2), J?.2 (Pin_2), J?.2 (Pin_2), J?.2 (Pin_2), J?.2 (Pin_2)
- new net GND: J?.1 (Pin_1)
- new net SCL: J?.4 (Pin_4)
- new net SDA: J?.3 (Pin_3)
- new net VCC: J?.2 (Pin_2)
