File: MCU.sch (KiCad schematic (older format))
At the start: 9 parts

Commit message: Completed Initial Schematic
Parts:
- added J?: ICSP, symbol Connector_Generic:Conn_02x03_Odd_Even
- added R? (x2): 1.2K, symbol Device:R
- U?: symbol MCU_Microchip_ATmega:ATmega328P-AU -> 3d_Printer_Interface-rescue:ATmega328P-AU-MCU_Microchip_ATmega
Connections:
- net +5V: now also J?.2 (Pin_2), R?.1, R?.1
- net D11: now also J?.4 (Pin_4)
- net D12: now also J?.1 (Pin_1)
- net D13: now also J?.3 (Pin_3)
- net GND: now also J?.6 (Pin_6)
- net MCU_RESET: now also J?.5 (Pin_5)
- net AD4 renamed SDA
- net SDA: now also R?.2
- net AD5 renamed SCL
- net SCL: now also R?.2
Other:
- moved on the sheet: R?, U?, Y?
