File: USB_Serial.sch (KiCad schematic (older format))
At the start: 9 parts

Commit message: Completed Initial Schematic
Parts:
- added D?: TX_LED, symbol Device:LED
- added D?: RX_LED, symbol Device:LED
- added R? (x2): 470, symbol Device:R
- R?: value 4.7k -> 470
- U?: symbol Interface_USB:FT232RL -> 3d_Printer_Interface-rescue:FT232RL-Interface_USB
Connections:
- net +5V: now also R?.1, R?.1
- net at U?.22 (CBUS1): now also D?.1 (K)
- net at U?.23 (CBUS0): now also D?.1 (K)
- new net: D?.2 (A), R?.2 (x2)
- no-connect marks 13 -> 11
Other:
- moved on the sheet: D?, R?
Changed lines of the file:
@@
 $Descr A4 11693 8268
 encoding utf-8
-Sheet 2 3
+Sheet 2 9
 Title ""
 Date ""
@@
 $EndDescr
 $Comp
-L Interface_USB:FT232RL U?
+L 3d_Printer_Interface-rescue:FT232RL-Interface_USB U?
 U 1 1 5E37E418
 P 5000 3450
+AR Path="/5E37E418" Ref="U?"  Part="1"
+AR Path="/5E37E377/5E37E418" Ref="U?"  Part="1"
 F 0 "U?" H 5000 4631 50  0000 C CNN
 F 1 "FT232RL" H 5000 4540 50  0000 C CNN
@@
 	5100 2450 5400 2450
 Wire Wire Line
-	5400 2450 5400 2100
+	5400 2450 5400 2250
 Connection ~ 5100 2450
 $Comp
@@
 L Device:LED D?
 U 1 1 5E3A74E8
-P 3050 3900
-F 0 "D?" V 3089 3782 50  0000 R CNN
-F 1 "PWR" V 2998 3782 50  0000 R CNN
-F 2 "" H 3050 3900 50  0001 C CNN
-F 3 "~" H 3050 3900 50  0001 C CNN
-	1    3050 3900
+P 8150 3450
+F 0 "D?" V 8189 3332 50  0000 R CNN
+F 1 "PWR" V 8098 3332 50  0000 R CNN
+F 2 "" H 8150 3450 50  0001 C CNN
+F 3 "~" H 8150 3450 50  0001 C CNN
+	1    8150 3450
 	0    -1   -1   0
 $EndComp
@@
 L Device:R R?
 U 1 1 5E3A806D
-P 3050 3450
-F 0 "R?" H 3120 3496 50  0000 L CNN
-F 1 "4.7k" H 3120 3405 50  0000 L CNN
-F 2 "" V 2980 3450 50  0001 C CNN
-F 3 "~" H 3050 3450 50  0001 C CNN
-	1    3050 3450
-	1    0    0    -1
-$EndComp
-Wire Wire Line
-	3050 3600 3050 3750
+P 8150 3000
+F 0 "R?" H 8220 3046 50  0000 L CNN
+F 1 "470" H 8220 2955 50  0000 L CNN
+F 2 "" V 8080 3000 50  0001 C CNN
+F 3 "~" H 8150 3000 50  0001 C CNN
+	1    8150 3000
+	1    0    0    -1
+$EndComp
+Wire Wire Line
+	8150 3150 8150 3300
 $Comp
 L power:GND #PWR?
 U 1 1 5E3A8DBA
-P 3050 4200
-F 0 "#PWR?" H 3050 3950 50  0001 C CNN
-F 1 "GND" H 3055 4027 50  0000 C CNN
-F 2 "" H 3050 4200 50  0001 C CNN
-F 3 "" H 3050 4200 50  0001 C CNN
-	1    3050 4200
+P 8150 3750
+F 0 "#PWR?" H 8150 3500 50  0001 C CNN
+F 1 "GND" H 8155 3577 50  0000 C CNN
+F 2 "" H 8150 3750 50  0001 C CNN
+F 3 "" H 8150 3750 50  0001 C CNN
+	1    8150 3750
 	1    0    0    -1
 $EndComp
@@
 L power:+5V #PWR?
 U 1 1 5E3A924B
-P 3050 3200
-F 0 "#PWR?" H 3050 3050 50  0001 C CNN
-F 1 "+5V" H 3065 3373 50  0000 C CNN
-F 2 "" H 3050 3200 50  0001 C CNN
-F 3 "" H 3050 3200 50  0001 C CNN
-	1    3050 3200
-	1    0    0    -1
-$EndComp
-Wire Wire Line
-	3050 4050 3050 4200
-Wire Wire Line
-	3050 3200 3050 3300
-NoConn ~ 5800 3750
-NoConn ~ 5800 3850
+P 8150 2750
+F 0 "#PWR?" H 8150 2600 50  0001 C CNN
+F 1 "+5V" H 8165 2923 50  0000 C CNN
+F 2 "" H 8150 2750 50  0001 C CNN
+F 3 "" H 8150 2750 50  0001 C CNN
+	1    8150 2750
+	1    0    0    -1
+$EndComp
+Wire Wire Line
+	8150 3600 8150 3750
+Wire Wire Line
+	8150 2750 8150 2850
 NoConn ~ 5800 3950
 NoConn ~ 5800 4050
@@
 NoConn ~ 5800 3350
 NoConn ~ 5800 3450
+$Comp
+L Device:LED D?
+U 1 1 5E3D6F1E
+P 7000 3450
+F 0 "D?" V 7039 3333 50  0000 R CNN
+F 1 "TX_LED" V 6948 3333 50  0000 R CNN
+F 2 "" H 7000 3450 50  0001 C CNN
+F 3 "~" H 7000 3450 50  0001 C CNN
+	1    7000 3450
+	0    -1   -1   0
+$EndComp
+$Comp
+L Device:LED D?
+U 1 1 5E3D7AA8
+P 7500 3450
+F 0 "D?" V 7539 3332 50  0000 R CNN
+F 1 "RX_LED" V 7448 3332 50  0000 R CNN
+F 2 "" H 7500 3450 50  0001 C CNN
+F 3 "~" H 7500 3450 50  0001 C CNN
+	1    7500 3450
+	0    -1   -1   0
+$EndComp
+$Comp
+L Device:R R?
+U 1 1 5E3D8216
+P 7000 3050
+F 0 "R?" H 7070 3096 50  0000 L CNN
+F 1 "470" H 7070 3005 50  0000 L CNN
+F 2 "" V 6930 3050 50  0001 C CNN
+F 3 "~" H 7000 3050 50  0001 C CNN
+	1    7000 3050
+	1    0    0    -1
+$EndComp
+$Comp
+L Device:R R?
+U 1 1 5E3D8516
+P 7500 3050
+F 0 "R?" H 7570 3096 50  0000 L CNN
+F 1 "470" H 7570 3005 50  0000 L CNN
+F 2 "" V 7430 3050 50  0001 C CNN
+F 3 "~" H 7500 3050 50  0001 C CNN
+	1    7500 3050
+	1    0    0    -1
+$EndComp
+Wire Wire Line
+	7000 3200 7000 3300
+Wire Wire Line
+	7000 3600 7000 3750
+Wire Wire Line
+	7000 3750 5800 3750
+Wire Wire Line
+	5800 3850 7500 3850
+Wire Wire Line
+	7500 3850 7500 3600
+Wire Wire Line
+	7500 3300 7500 3200
+Wire Wire Line
+	5400 2250 7000 2250
+Wire Wire Line
+	7000 2250 7000 2900
+Connection ~ 5400 2250
+Wire Wire Line
+	5400 2250 5400 2100
+Wire Wire Line
+	7500 2900 7500 2250
+Wire Wire Line
+	7500 2250 7000 2250
+Connection ~ 7000 2250
 $EndSCHEMATC
